File: attiny_rfid_lightbackup11122020.kicad_pcb (KiCad board)
At the start: 2 copper layers, 75 x 99.1 mm, 30 parts, among them IC1 EM4095, U1 ESP32-WROOM-32, U2 NCP1117-3.3_SOT223, m2 MountingHole_2.1mm

Commit message: updated values to match place values
Parts:
- C_RESOptional1: value 220pf but 300 would be better -> NA
Connections:
- net /EN renamed Net-(C1-Pad2)
- net /IO0 renamed Net-(J_DEBUG1-Pad7)
- net /RX renamed Net-(J_DEBUG1-Pad5)
- net /TX renamed Net-(J_DEBUG1-Pad6)
