File: attiny_rfid_light.kicad_pcb (KiCad board)
At the start: 2 copper layers, 75 x 99.1 mm, 30 parts, among them IC1 EM4095, U1 ESP32-WROOM-32, U2 NCP1117-3.3_SOT223, m2 MountingHole_2.1mm

Commit message: v4
Parts:
- removed J_DEBUG1: Conn_01x08_Male, Connector_PinHeader_2.54mm:PinHeader_1x08_P2.54mm_Vertical
- added C_RESC1: optional, Capacitor_SMD:C_0805_2012Metric_Pad1.18x1.45mm_HandSolder, F.Cu at (137.1, 139.6)
- added J1: Conn_01x16_Male, Connector_PinHeader_2.54mm:PinHeader_1x16_P2.54mm_Vertical, F.Cu at (96.5, 152.4)
- added RMOD1: 10k, Resistor_SMD:R_0805_2012Metric_Pad1.20x1.40mm_HandSolder, F.Cu at (120.5, 145.4)
- C_Big1: footprint Capacitor_THT:C_Radial_D5.0mm_H11.0mm_P2.00mm -> Capacitor_SMD:CP_Elec_8x10.5
- C_RESB1: renamed from C_RESOptional1; value 220pf but 300 would be better -> 300pf
- J_POWER1: footprint Connector_USB:USB_Micro-B_Molex-105017-0001 -> Connector_USB:USB_Micro-B_Molex_47346-0001
- R_2: value 5k1 or 5k? was 5k og -> 5k1
- R_4: value 5k1 og was 5k -> 5k1
- moved C_REG1 27.6 mm to (97.8, 148.0), turned to 180 degrees
- moved C_Big1 26.7 mm to (110.3, 139.5), turned to -90 degrees
- moved U2 22.7 mm to (100.0, 141.7), turned to 90 degrees
- moved JLED1 22.2 mm to (97.8, 132.2)
- moved R_3 21.1 mm to (105.9, 133.0), turned to -90 degrees
- moved R_4 18.0 mm to (69.4, 135.9), turned to 180 degrees
- moved U1 17.4 mm to (83.8, 144.8)
- moved C_REG2 16.4 mm to (103.3, 148.1)
- moved R_2 7.88 mm to (95.2, 138.2), turned to 90 degrees
- moved C_RESB1 7.76 mm to (137.2, 136.4)
- moved C_RESA1 5.18 mm to (137.2, 133.0)
- moved C_DEC1 4.97 mm to (125.1, 145.4), turned to 0 degrees
- moved R_1 4.78 mm to (120.5, 142.2)
- moved C2 4.64 mm to (120.5, 138.7)
- moved C_AGND1 1.93 mm to (129.4, 145.4)
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- renumbered C_DV1 to C_REG1, C_DV2 to C_REG2, C_RES1 to C_RESA1, m2 to m2a, m2 to m2b, m2 to m2c, m2 to m2d
Connections:
- net Net-(IC1-Pad13) renamed /DEMOD_OUT
- net Net-(IC1-Pad14) renamed /SHD
- net Net-(IC1-Pad2) renamed /RDY_CLK
- IC1 pad 12: GND -> /MOD
- U1 pad 10: unconnected-(U1-Pad10) -> /25
- U1 pad 11: unconnected-(U1-Pad11) -> /26
- U1 pad 12: unconnected-(U1-Pad12) -> /MOD
- U1 pad 29: Net-(J_DEBUG1-Pad4) -> /5
- U1 pad 30: unconnected-(U1-Pad30) -> /18
- U1 pad 31: unconnected-(U1-Pad31) -> /19
- U1 pad 33: unconnected-(U1-Pad33) -> /21
- U1 pad 36: unconnected-(U1-Pad36) -> /22
- U1 pad 8: unconnected-(U1-Pad8) -> /32
- U1 pad 9: unconnected-(U1-Pad9) -> /33
Routing:
- net /18: track 0.00 -> 53.3 mm, vias 0 -> 1
- net /19: track 0.00 -> 50.4 mm, vias 0 -> 1
- net /32: track 0.00 -> 48.5 mm, vias 0 -> 1
- net /21: track 0.00 -> 47.1 mm, vias 0 -> 1
- net /MOD: track 0.00 -> 46.4 mm
- net /33: track 0.00 -> 44.8 mm, vias 0 -> 1
- net /22: track 0.00 -> 44.1 mm
- net /26: track 0.00 -> 42.4 mm, vias 0 -> 1
- net /25: track 0.00 -> 39.4 mm, vias 0 -> 1
- net Net-(J_DEBUG1-Pad4): track 37.8 -> 0.00 mm, vias 1 -> 0
- net /5: track 0.00 -> 35.4 mm
- net /SHD: track 45.5 -> 69.0 mm
- net +3V3: track 85.3 -> 64.0 mm, vias 1 -> 0
- net /IO0: track 50.1 -> 70.7 mm, vias 1 -> 2
- net /EN: track 37.2 -> 55.3 mm
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
Commit message: v5
Parts:
- C_DV4: value 3.7nf split between 2 -> 3.6nf
- C_DV5: value 3.7nf split between 2 -> optional
- C_RESB1: value 300pf -> 470pf
- RMOD1: value 10k -> 12k
Changed lines of the file:
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@@
       (effects (font (size 1 1) (thickness 0.15)))
     )
-    (fp_text value "3.7nf split between 2" (at 0 1.68) (layer "F.Fab")
+    (fp_text value "optional" (at 0 1.68) (layer "F.Fab")
       (effects (font (size 1 1) (thickness 0.15)))
     )
@@
       (effects (font (size 1 1) (thickness 0.15)))
     )
-    (fp_text value "3.7nf split between 2" (at 0 1.68) (layer "F.Fab")
+    (fp_text value "3.6nf" (at 0 1.68) (layer "F.Fab")
       (effects (font (size 1 1) (thickness 0.15)))
     )
@@
       (effects (font (size 1 1) (thickness 0.15)))
     )
-    (fp_text value "300pf" (at 0 1.68) (layer "F.Fab")
+    (fp_text value "470pf" (at 0 1.68) (layer "F.Fab")
       (effects (font (size 1 1) (thickness 0.15)))
     )
@@
       (effects (font (size 1 1) (thickness 0.15)))
     )
-    (fp_text value "10k" (at 0 1.65) (layer "F.Fab")
-      (effects (font (size 1 1) (thickness 0.15)))
-    )
+    (fp_text value "12k" (at 0 1.65) (layer "F.Fab")
+      (effects (font (size 1 1) (thickness 0.15)))
+    )
